Commit message: Add markers to model wheels to make rotation visual tracking easier

File: smallbot_description/urdf/smallbot.xacro (robot description, xacro)
@@ -62,4 +62,13 @@
         </collision>
     </link>
+    <link name="rear_left_wheel_marker">
+        <visual>
+            <origin xyz="0 0 0" rpy="0 0 0" />
+            <geometry>
+                <box size="0.03 0.005 0.005" />
+            </geometry>
+            <material name="White" />
+        </visual>
+    </link>
     <link name="rear_right_wheel">
         <visual>
@@ -77,4 +86,13 @@
         </collision>
     </link>
+        <link name="rear_right_wheel_marker">
+        <visual>
+            <origin xyz="0 0 0" rpy="0 0 0" />
+            <geometry>
+                <box size="0.03 0.005 0.005" />
+            </geometry>
+            <material name="White" />
+        </visual>
+    </link>
     <link name="front_left_wheel">
         <visual>
@@ -92,4 +110,13 @@
         </collision>
     </link>
+    <link name="front_left_wheel_marker">
+        <visual>
+            <origin xyz="0 0 0" rpy="0 0 0" />
+            <geometry>
+                <box size="0.03 0.005 0.005" />
+            </geometry>
+            <material name="White" />
+        </visual>
+    </link>
     <link name="front_right_wheel">
         <visual>
@@ -107,4 +134,13 @@
         </collision>
     </link>
+        <link name="front_right_wheel_marker">
+        <visual>
+            <origin xyz="0 0 0" rpy="0 0 0" />
+            <geometry>
+                <box size="0.03 0.005 0.005" />
+            </geometry>
+            <material name="White" />
+        </visual>
+    </link>
     <link name="middle_left_wheel">
         <visual>
@@ -122,4 +158,13 @@
         </collision>
     </link>
+        <link name="middle_left_wheel_marker">
+        <visual>
+            <origin xyz="0 0 0" rpy="0 0 0" />
+            <geometry>
+                <box size="0.03 0.005 0.005" />
+            </geometry>
+            <material name="White" />
+        </visual>
+    </link>
     <link name="middle_right_wheel">
         <visual>
@@ -136,4 +181,13 @@
             </geometry>
         </collision>
+    </link>
+    <link name="middle_right_wheel_marker">
+        <visual>
+            <origin xyz="0 0 0" rpy="0 0 0" />
+            <geometry>
+                <box size="0.03 0.005 0.005" />
+            </geometry>
+            <material name="White" />
+        </visual>
     </link>
     <joint name="base_to_rear_left_wheel" type="continuous">
@@ -143,4 +197,9 @@
         <origin xyz="-0.104 0.0925 0" rpy="0 0 0"/>
     </joint>
+    <joint name="rear_left_wheel_to_marker" type="fixed">
+        <parent link="rear_left_wheel" />
+        <child link="rear_left_wheel_marker" />
+        <origin xyz="0.015 0.0175 0" rpy="0 0 0" />
+    </joint>
     <joint name="base_to_rear_right_wheel" type="continuous">
         <axis rpy="0 0 0" xyz="0 1 0"/>
@@ -149,4 +208,9 @@
 		<origin xyz="-0.104 -0.0925 0" rpy="0 0 0"/>
     </joint>
+    <joint name="rear_right_wheel_to_marker" type="fixed">
+        <parent link="rear_right_wheel" />
+        <child link="rear_right_wheel_marker" />
+        <origin xyz="0.015 -0.0175 0" rpy="0 0 0" />
+    </joint>
     <joint name="base_to_front_left_wheel" type="continuous">
         <axis rpy="0 0 0" xyz="0 1 0"/>
@@ -155,4 +219,9 @@
 		<origin xyz="0.104 0.0925 0" rpy="0 0 0" />
     </joint>
+    <joint name="front_left_wheel_to_marker" type="fixed">
+        <parent link="front_left_wheel" />
+        <child link="front_left_wheel_marker" />
+        <origin xyz="0.015 0.0175 0" rpy="0 0 0" />
+    </joint>
     <joint name="base_to_front_right_wheel" type="continuous">
         <axis rpy="0 0 0" xyz="0 1 0"/>
@@ -161,4 +230,9 @@
 		<origin xyz="0.104 -0.0925 0" rpy="0 0 0" />
     </joint>
+    <joint name="front_right_wheel_to_marker" type="fixed">
+        <parent link="front_right_wheel" />
+        <child link="front_right_wheel_marker" />
+        <origin xyz="0.015 -0.0175 0" rpy="0 0 0" />
+    </joint>
     <joint name="base_to_middle_left_wheel" type="continuous">
         <axis rpy="0 0 0" xyz="0 1 0"/>
@@ -167,4 +241,9 @@
 		<origin xyz="0 0.0925 0" rpy="0 0 0" />
     </joint>
+    <joint name="middle_left_wheel_to_marker" type="fixed">
+        <parent link="middle_left_wheel" />
+        <child link="middle_left_wheel_marker" />
+        <origin xyz="0.015 0.0175 0" rpy="0 0 0" />
+    </joint>
     <joint name="base_to_middle_right_wheel" type="continuous">
         <axis rpy="0 0 0" xyz="0 1 0"/>
@@ -173,3 +252,8 @@
 		<origin xyz="0 -0.0925 0" rpy="0 0 0" />
     </joint>
+    <joint name="middle_right_wheel_to_marker" type="fixed">
+        <parent link="middle_right_wheel" />
+        <child link="middle_right_wheel_marker" />
+        <origin xyz="0.015 -0.0175 0" rpy="0 0 0" />
+    </joint>
 </robot>

Commit message: Adopt model for use with controller

File: smallbot_description/urdf/smallbot.xacro (robot description, xacro)
@@ -5,4 +5,8 @@
 	<xacro:include filename="$(find smallbot_description)/urdf/smallbot_materials.xacro" />
     <xacro:property name="clearance" value="0.035" />
+    <xacro:property name="wheel_radius" value="0.035"/>
+    <xacro:property name="wheel_separation" value="0.15"/>
+    <xacro:property name="wheel_width" value="0.035"/>
+    <xacro:property name="PI" value="3.1415926"/>
 	<!-- abot_base -->
 	<link name="base_link">
@@ -15,5 +19,5 @@
 			<origin xyz="0 0 0.03" rpy="0 0 0" />
             <geometry>
-                <box size="0.28 0.15 0.08"/>
+                <box size="0.28 ${wheel_separation} 0.08"/>
             </geometry>
 			<material name="White" />
@@ -22,5 +26,5 @@
 			<origin xyz="0 0 0.03" rpy="0 0 0" />
             <geometry>
-                <box size="0.28 0.15 0.08"/>
+                <box size="0.28 ${wheel_separation} 0.08"/>
             </geometry>
 		</collision>
@@ -37,5 +41,5 @@
             <origin xyz="0 0 0" rpy="0 0 0" />
             <geometry>
-                <box size="0.28 0.22 0.001"/>
+                <box size="0.28 ${wheel_separation + wheel_width + wheel_width} 0.001"/>
             </geometry>
             <material name="Blue" />
@@ -51,12 +55,12 @@
 			<origin xyz="0 0 0" rpy="1.5708 0 0" />
             <geometry>
-                <cylinder length="0.035" radius="0.035"/>
-            </geometry>
-            <material name="Red" />
-        </visual>
-        <collision>
-			<origin xyz="0 0 0" rpy="1.5708 0 0" />
-            <geometry>
-                <cylinder length="0.035" radius="0.035"/>
+                <cylinder length="${wheel_width}" radius="${wheel_radius}"/>
+            </geometry>
+            <material name="Red" />
+        </visual>
+        <collision>
+			<origin xyz="0 0 0" rpy="1.5708 0 0" />
+            <geometry>
+                <cylinder length="${wheel_width}" radius="${wheel_radius}"/>
             </geometry>
         </collision>
@@ -75,12 +79,12 @@
 			<origin xyz="0 0 0" rpy="1.5708 0 0" />
             <geometry>
-                <cylinder length="0.035" radius="0.035"/>
-            </geometry>
-            <material name="Red" />
-        </visual>
-        <collision>
-			<origin xyz="0 0 0" rpy="1.5708 0 0" />
-            <geometry>
-                <cylinder length="0.035" radius="0.035"/>
+                <cylinder length="${wheel_width}" radius="${wheel_radius}"/>
+            </geometry>
+            <material name="Red" />
+        </visual>
+        <collision>
+			<origin xyz="0 0 0" rpy="1.5708 0 0" />
+            <geometry>
+                <cylinder length="${wheel_width}" radius="${wheel_radius}"/>
             </geometry>
         </collision>
@@ -99,12 +103,12 @@
 			<origin xyz="0 0 0" rpy="1.5708 0 0" />
             <geometry>
-                <cylinder length="0.035" radius="0.035"/>
-            </geometry>
-            <material name="Red" />
-        </visual>
-        <collision>
-			<origin xyz="0 0 0" rpy="1.5708 0 0" />
-            <geometry>
-                <cylinder length="0.035" radius="0.035"/>
+                <cylinder length="${wheel_width}" radius="${wheel_radius}"/>
+            </geometry>
+            <material name="Red" />
+        </visual>
+        <collision>
+			<origin xyz="0 0 0" rpy="1.5708 0 0" />
+            <geometry>
+                <cylinder length="${wheel_width}" radius="${wheel_radius}"/>
             </geometry>
         </collision>
@@ -123,12 +127,12 @@
 			<origin xyz="0 0 0" rpy="1.5708 0 0" />
             <geometry>
-                <cylinder length="0.035" radius="0.035"/>
-            </geometry>
-            <material name="Red" />
-        </visual>
-        <collision>
-			<origin xyz="0 0 0" rpy="1.5708 0 0" />
-            <geometry>
-                <cylinder length="0.035" radius="0.035"/>
+                <cylinder length="${wheel_width}" radius="${wheel_radius}"/>
+            </geometry>
+            <material name="Red" />
+        </visual>
+        <collision>
+			<origin xyz="0 0 0" rpy="1.5708 0 0" />
+            <geometry>
+                <cylinder length="${wheel_width}" radius="${wheel_radius}"/>
             </geometry>
         </collision>
@@ -147,12 +151,12 @@
 			<origin xyz="0 0 0" rpy="1.5708 0 0" />
             <geometry>
-                <cylinder length="0.035" radius="0.035"/>
-            </geometry>
-            <material name="Red" />
-        </visual>
-        <collision>
-			<origin xyz="0 0 0" rpy="1.5708 0 0" />
-            <geometry>
-                <cylinder length="0.035" radius="0.035"/>
+                <cylinder length="${wheel_width}" radius="${wheel_radius}"/>
+            </geometry>
+            <material name="Red" />
+        </visual>
+        <collision>
+			<origin xyz="0 0 0" rpy="1.5708 0 0" />
+            <geometry>
+                <cylinder length="${wheel_width}" radius="${wheel_radius}"/>
             </geometry>
         </collision>
@@ -171,12 +175,12 @@
 			<origin xyz="0 0 0" rpy="1.5708 0 0" />
             <geometry>
-                <cylinder length="0.035" radius="0.035"/>
-            </geometry>
-            <material name="Red" />
-        </visual>
-        <collision>
-			<origin xyz="0 0 0" rpy="1.5708 0 0" />
-            <geometry>
-                <cylinder length="0.035" radius="0.035"/>
+                <cylinder length="${wheel_width}" radius="${wheel_radius}"/>
+            </geometry>
+            <material name="Red" />
+        </visual>
+        <collision>
+			<origin xyz="0 0 0" rpy="1.5708 0 0" />
+            <geometry>
+                <cylinder length="${wheel_width}" radius="${wheel_radius}"/>
             </geometry>
         </collision>
@@ -195,5 +199,5 @@
         <parent link="base_link" />
         <child link="rear_left_wheel" />
-        <origin xyz="-0.104 0.0925 0" rpy="0 0 0"/>
+        <origin xyz="-0.104 ${wheel_separation/2 + wheel_width/2} 0" rpy="0 0 0"/>
     </joint>
     <joint name="rear_left_wheel_to_marker" type="fixed">
@@ -206,5 +210,5 @@
         <parent link="base_link" />
         <child link="rear_right_wheel" />
-		<origin xyz="-0.104 -0.0925 0" rpy="0 0 0"/>
+		<origin xyz="-0.104 ${-1 * (wheel_separation/2 + wheel_width/2)} 0" rpy="0 0 0"/>
     </joint>
     <joint name="rear_right_wheel_to_marker" type="fixed">
@@ -217,5 +221,5 @@
         <parent link="base_link" />
         <child link="front_left_wheel" />
-		<origin xyz="0.104 0.0925 0" rpy="0 0 0" />
+		<origin xyz="0.104 ${wheel_separation/2 + wheel_width/2} 0" rpy="0 0 0" />
     </joint>
     <joint name="front_left_wheel_to_marker" type="fixed">
@@ -228,5 +232,5 @@
         <parent link="base_link" />
         <child link="front_right_wheel" />
-		<origin xyz="0.104 -0.0925 0" rpy="0 0 0" />
+		<origin xyz="0.104 ${-1 * (wheel_separation/2 + wheel_width/2)} 0" rpy="0 0 0" />
     </joint>
     <joint name="front_right_wheel_to_marker" type="fixed">
@@ -239,5 +243,5 @@
         <parent link="base_link" />
         <child link="middle_left_wheel" />
-		<origin xyz="0 0.0925 0" rpy="0 0 0" />
+		<origin xyz="0 ${wheel_separation/2 + wheel_width/2} 0" rpy="0 0 0" />
     </joint>
     <joint name="middle_left_wheel_to_marker" type="fixed">
@@ -250,5 +254,5 @@
         <parent link="base_link" />
         <child link="middle_right_wheel" />
-		<origin xyz="0 -0.0925 0" rpy="0 0 0" />
+		<origin xyz="0 ${-1 * (wheel_separation/2 + wheel_width/2)} 0" rpy="0 0 0" />
     </joint>
     <joint name="middle_right_wheel_to_marker" type="fixed">
