Commit message: Finished gazebo simulation

File: smallbot_description/urdf/smallbot.xacro (robot description, xacro)
@@ -4,16 +4,25 @@
 	<!-- Matherials -->
 	<xacro:include filename="$(find smallbot_description)/urdf/smallbot_materials.xacro" />
+    <!-- Gazebo parameters -->
+    <xacro:include filename="$(find smallbot_description)/urdf/smallbot.gazebo" />
     <xacro:property name="clearance" value="0.035" />
     <xacro:property name="wheel_radius" value="0.035"/>
     <xacro:property name="wheel_separation" value="0.15"/>
     <xacro:property name="wheel_width" value="0.035"/>
+    <xacro:property name="mass" value="0.1"/>
+    <xacro:property name="wheel_mass" value="0.2"/>
+    <xacro:property name="marker_mass" value="0.0"/>
+    <xacro:property name="inertia" value="1.0"/>
     <xacro:property name="PI" value="3.1415926"/>
-	<!-- abot_base -->
-	<link name="base_link">
-		<!-- <inertial>
-			<origin xyz="0 0 0.07" rpy="0 0 0" />
-			<mass value="0.27459"/>
-			<inertia ixx="0.00032396" ixy="-1.1142E-12" ixz="-9.1302E-06" iyy="0.00030091" iyz="-3.3253E-10" izz="0.00056103"/>
-		</inertial> -->
+    <xacro:property name="wheel_ixx" value="${wheel_mass*(3*wheel_radius*wheel_radius+wheel_width*wheel_width)/12}" />
+    <xacro:property name="wheel_ixy" value="0.0" />
+    <xacro:property name="wheel_ixz" value="0.0" />
+    <xacro:property name="wheel_iyy" value="${wheel_mass*(3*wheel_radius*wheel_radius+wheel_width*wheel_width)/12}" />
+    <xacro:property name="wheel_iyz" value="0.0" />
+    <xacro:property name="wheel_izz" value="${wheel_mass*wheel_radius*wheel_radius/2}" />
+	<!-- smallbot_base -->
+    <link name="base_link">
+    </link>
+	<link name="body_link">
 		<visual>
 			<origin xyz="0 0 0.03" rpy="0 0 0" />
@@ -29,40 +38,34 @@
             </geometry>
 		</collision>
-		<!-- <collision>
-			<origin xyz="0 0 0" rpy="0 0 0" />
-			<geometry>
-				<mesh filename="package://abot_description/meshes/abot_base.STL" />
-			</geometry>
-		</collision> -->
+        <inertial>
+            <origin xyz="0 0 0.03" rpy="0 0 0" />
+            <mass value="${mass}" />
+            <inertia ixx="${inertia}" ixy="0.0" ixz="0.0" iyy="${inertia}" iyz="0.0" izz="${inertia}" />
+        </inertial>
 	</link>
-    <!-- base_footprint -->
-    <link name="base_footprint">
-        <visual>
-            <origin xyz="0 0 0" rpy="0 0 0" />
-            <geometry>
-                <box size="0.28 ${wheel_separation + wheel_width + wheel_width} 0.001"/>
-            </geometry>
-            <material name="Blue" />
-        </visual>
-    </link>
-    <joint name="base_footprint_to_base_link" type="fixed">
-        <origin xyz="0 0 ${clearance}" rpy="0 0 0" />
-        <parent link="base_footprint" />
-        <child link="base_link" />
+    <joint name="base_to_body" type="fixed">
+        <axis rpy="0 0 0" xyz="0 0 0"/>
+        <parent link="base_link" />
+        <child link="body_link" />
+        <origin xyz="0 0 ${wheel_radius}" rpy="0 0 0"/>
     </joint>
     <link name="rear_left_wheel">
         <visual>
-			<origin xyz="0 0 0" rpy="1.5708 0 0" />
-            <geometry>
-                <cylinder length="${wheel_width}" radius="${wheel_radius}"/>
-            </geometry>
-            <material name="Red" />
-        </visual>
-        <collision>
-			<origin xyz="0 0 0" rpy="1.5708 0 0" />
-            <geometry>
-                <cylinder length="${wheel_width}" radius="${wheel_radius}"/>
-            </geometry>
-        </collision>
+			<origin xyz="0 0 0" rpy="${PI / 2} 0 0" />
+            <geometry>
+                <cylinder length="${wheel_width}" radius="${wheel_radius}"/>
+            </geometry>
+            <material name="Red" />
+        </visual>
+        <collision>
+			<origin xyz="0 0 0" rpy="${PI / 2} 0 0" />
+            <geometry>
+                <cylinder length="${wheel_width}" radius="${wheel_radius}"/>
+            </geometry>
+        </collision>
+        <inertial>
+            <mass value="${wheel_mass}" />
+            <inertia ixx="${wheel_ixx}" ixy="${wheel_ixy}" ixz="${wheel_ixz}" iyy="${wheel_iyy}" iyz="${wheel_iyz}" izz="${wheel_izz}" />
+        </inertial>
     </link>
     <link name="rear_left_wheel_marker">
@@ -74,43 +77,59 @@
             <material name="White" />
         </visual>
+        <inertial>
+            <mass value="${marker_mass}" />
+            <inertia ixx="0.0" ixy="0.0" ixz="0.0" iyy="0.0" iyz="0.0" izz="0.0" />
+        </inertial>
     </link>
     <link name="rear_right_wheel">
         <visual>
-			<origin xyz="0 0 0" rpy="1.5708 0 0" />
-            <geometry>
-                <cylinder length="${wheel_width}" radius="${wheel_radius}"/>
-            </geometry>
-            <material name="Red" />
-        </visual>
-        <collision>
-			<origin xyz="0 0 0" rpy="1.5708 0 0" />
-            <geometry>
-                <cylinder length="${wheel_width}" radius="${wheel_radius}"/>
-            </geometry>
-        </collision>
-    </link>
-        <link name="rear_right_wheel_marker">
-        <visual>
-            <origin xyz="0 0 0" rpy="0 0 0" />
-            <geometry>
-                <box size="0.03 0.005 0.005" />
-            </geometry>
-            <material name="White" />
-        </visual>
+			<origin xyz="0 0 0" rpy="${PI / 2} 0 0" />
+            <geometry>
+                <cylinder length="${wheel_width}" radius="${wheel_radius}"/>
+            </geometry>
+            <material name="Red" />
+        </visual>
+        <collision>
+			<origin xyz="0 0 0" rpy="${PI / 2} 0 0" />
+            <geometry>
+                <cylinder length="${wheel_width}" radius="${wheel_radius}"/>
+            </geometry>
+        </collision>
+        <inertial>
+            <mass value="${wheel_mass}" />
+            <inertia ixx="${wheel_ixx}" ixy="${wheel_ixy}" ixz="${wheel_ixz}" iyy="${wheel_iyy}" iyz="${wheel_iyz}" izz="${wheel_izz}" />
+        </inertial>
+    </link>
+    <link name="rear_right_wheel_marker">
+        <visual>
+            <origin xyz="0 0 0" rpy="0 0 0" />
+            <geometry>
+                <box size="0.03 0.005 0.005" />
+            </geometry>
+            <material name="White" />
+        </visual>
+        <inertial>
+            <mass value="${marker_mass}" />
+            <inertia ixx="0.0" ixy="0.0" ixz="0.0" iyy="0.0" iyz="0.0" izz="0.0" />
+        </inertial>
     </link>
     <link name="front_left_wheel">
         <visual>
-			<origin xyz="0 0 0" rpy="1.5708 0 0" />
-            <geometry>
-                <cylinder length="${wheel_width}" radius="${wheel_radius}"/>
-            </geometry>
-            <material name="Red" />
-        </visual>
-        <collision>
-			<origin xyz="0 0 0" rpy="1.5708 0 0" />
-            <geometry>
-                <cylinder length="${wheel_width}" radius="${wheel_radius}"/>
-            </geometry>
-        </collision>
+			<origin xyz="0 0 0" rpy="${PI / 2} 0 0" />
+            <geometry>
+                <cylinder length="${wheel_width}" radius="${wheel_radius}"/>
+            </geometry>
+            <material name="Red" />
+        </visual>
+        <collision>
+			<origin xyz="0 0 0" rpy="${PI / 2} 0 0" />
+            <geometry>
+                <cylinder length="${wheel_width}" radius="${wheel_radius}"/>
+            </geometry>
+        </collision>
+        <inertial>
+            <mass value="${wheel_mass}" />
+            <inertia ixx="${wheel_ixx}" ixy="${wheel_ixy}" ixz="${wheel_ixz}" iyy="${wheel_iyy}" iyz="${wheel_iyz}" izz="${wheel_izz}" />
+        </inertial>
     </link>
     <link name="front_left_wheel_marker">
@@ -122,67 +141,91 @@
             <material name="White" />
         </visual>
+        <inertial>
+            <mass value="${marker_mass}" />
+            <inertia ixx="0.0" ixy="0.0" ixz="0.0" iyy="0.0" iyz="0.0" izz="0.0" />
+        </inertial>
     </link>
     <link name="front_right_wheel">
         <visual>
-			<origin xyz="0 0 0" rpy="1.5708 0 0" />
-            <geometry>
-                <cylinder length="${wheel_width}" radius="${wheel_radius}"/>
-            </geometry>
-            <material name="Red" />
-        </visual>
-        <collision>
-			<origin xyz="0 0 0" rpy="1.5708 0 0" />
-            <geometry>
-                <cylinder length="${wheel_width}" radius="${wheel_radius}"/>
-            </geometry>
-        </collision>
-    </link>
-        <link name="front_right_wheel_marker">
-        <visual>
-            <origin xyz="0 0 0" rpy="0 0 0" />
-            <geometry>
-                <box size="0.03 0.005 0.005" />
-            </geometry>
-            <material name="White" />
-        </visual>
+			<origin xyz="0 0 0" rpy="${PI / 2} 0 0" />
+            <geometry>
+                <cylinder length="${wheel_width}" radius="${wheel_radius}"/>
+            </geometry>
+            <material name="Red" />
+        </visual>
+        <collision>
+			<origin xyz="0 0 0" rpy="${PI / 2} 0 0" />
+            <geometry>
+                <cylinder length="${wheel_width}" radius="${wheel_radius}"/>
+            </geometry>
+        </collision>
+        <inertial>
+            <mass value="${wheel_mass}" />
+            <inertia ixx="${wheel_ixx}" ixy="${wheel_ixy}" ixz="${wheel_ixz}" iyy="${wheel_iyy}" iyz="${wheel_iyz}" izz="${wheel_izz}" />
+        </inertial>
+    </link>
+    <link name="front_right_wheel_marker">
+        <visual>
+            <origin xyz="0 0 0" rpy="0 0 0" />
+            <geometry>
+                <box size="0.03 0.005 0.005" />
+            </geometry>
+            <material name="White" />
+        </visual>
+        <inertial>
+            <mass value="${marker_mass}" />
+            <inertia ixx="0.0" ixy="0.0" ixz="0.0" iyy="0.0" iyz="0.0" izz="0.0" />
+        </inertial>
     </link>
     <link name="middle_left_wheel">
         <visual>
-			<origin xyz="0 0 0" rpy="1.5708 0 0" />
-            <geometry>
-                <cylinder length="${wheel_width}" radius="${wheel_radius}"/>
-            </geometry>
-            <material name="Red" />
-        </visual>
-        <collision>
-			<origin xyz="0 0 0" rpy="1.5708 0 0" />
-            <geometry>
-                <cylinder length="${wheel_width}" radius="${wheel_radius}"/>
-            </geometry>
-        </collision>
-    </link>
-        <link name="middle_left_wheel_marker">
-        <visual>
-            <origin xyz="0 0 0" rpy="0 0 0" />
-            <geometry>
-                <box size="0.03 0.005 0.005" />
-            </geometry>
-            <material name="White" />
-        </visual>
+			<origin xyz="0 0 0" rpy="${PI / 2} 0 0" />
+            <geometry>
+                <cylinder length="${wheel_width}" radius="${wheel_radius}"/>
+            </geometry>
+            <material name="Red" />
+        </visual>
+        <collision>
+			<origin xyz="0 0 0" rpy="${PI / 2} 0 0" />
+            <geometry>
+                <cylinder length="${wheel_width}" radius="${wheel_radius}"/>
+            </geometry>
+        </collision>
+        <inertial>
+            <mass value="${wheel_mass}" />
+            <inertia ixx="${wheel_ixx}" ixy="${wheel_ixy}" ixz="${wheel_ixz}" iyy="${wheel_iyy}" iyz="${wheel_iyz}" izz="${wheel_izz}" />
+        </inertial>
+    </link>
+    <link name="middle_left_wheel_marker">
+        <visual>
+            <origin xyz="0 0 0" rpy="0 0 0" />
+            <geometry>
+                <box size="0.03 0.005 0.005" />
+            </geometry>
+            <material name="White" />
+        </visual>
+        <inertial>
+            <mass value="${marker_mass}" />
+            <inertia ixx="0.0" ixy="0.0" ixz="0.0" iyy="0.0" iyz="0.0" izz="0.0" />
+        </inertial>
     </link>
     <link name="middle_right_wheel">
         <visual>
-			<origin xyz="0 0 0" rpy="1.5708 0 0" />
-            <geometry>
-                <cylinder length="${wheel_width}" radius="${wheel_radius}"/>
-            </geometry>
-            <material name="Red" />
-        </visual>
-        <collision>
-			<origin xyz="0 0 0" rpy="1.5708 0 0" />
-            <geometry>
-                <cylinder length="${wheel_width}" radius="${wheel_radius}"/>
-            </geometry>
-        </collision>
+			<origin xyz="0 0 0" rpy="${PI / 2} 0 0" />
+            <geometry>
+                <cylinder length="${wheel_width}" radius="${wheel_radius}"/>
+            </geometry>
+            <material name="Red" />
+        </visual>
+        <collision>
+			<origin xyz="0 0 0" rpy="${PI / 2} 0 0" />
+            <geometry>
+                <cylinder length="${wheel_width}" radius="${wheel_radius}"/>
+            </geometry>
+        </collision>
+        <inertial>
+            <mass value="${wheel_mass}" />
+            <inertia ixx="${wheel_ixx}" ixy="${wheel_ixy}" ixz="${wheel_ixz}" iyy="${wheel_iyy}" iyz="${wheel_iyz}" izz="${wheel_izz}" />
+        </inertial>
     </link>
     <link name="middle_right_wheel_marker">
@@ -194,10 +237,56 @@
             <material name="White" />
         </visual>
+        <inertial>
+            <mass value="${marker_mass}" />
+            <inertia ixx="0.0" ixy="0.0" ixz="0.0" iyy="0.0" iyz="0.0" izz="0.0" />
+        </inertial>
     </link>
     <joint name="base_to_rear_left_wheel" type="continuous">
         <axis rpy="0 0 0" xyz="0 1 0"/>
-        <parent link="base_link" />
+        <parent link="body_link" />
         <child link="rear_left_wheel" />
         <origin xyz="-0.104 ${wheel_separation/2 + wheel_width/2} 0" rpy="0 0 0"/>
+        <dynamics damping="0.0" friction="0.0"/>
+        <limit effort= "100" velocity="100"/>
+    </joint>
+    <joint name="base_to_rear_right_wheel" type="continuous">
+        <axis rpy="0 0 0" xyz="0 1 0"/>
+        <parent link="body_link" />
+        <child link="rear_right_wheel" />
+		<origin xyz="-0.104 ${-1 * (wheel_separation/2 + wheel_width/2)} 0" rpy="0 0 0"/>
+        <dynamics damping="0.0" friction="0.0"/>
+        <limit effort= "100" velocity="100"/>
+    </joint>
+    <joint name="base_to_front_left_wheel" type="continuous">
+        <axis rpy="0 0 0" xyz="0 1 0"/>
+        <parent link="body_link" />
+        <child link="front_left_wheel" />
+		<origin xyz="0.104 ${wheel_separation/2 + wheel_width/2} 0" rpy="0 0 0" />
+        <dynamics damping="0.0" friction="0.0"/>
+        <limit effort= "100" velocity="100"/>
+    </joint>
+    <joint name="base_to_front_right_wheel" type="continuous">
+        <axis rpy="0 0 0" xyz="0 1 0"/>
+        <parent link="body_link" />
+        <child link="front_right_wheel" />
+		<origin xyz="0.104 ${-1 * (wheel_separation/2 + wheel_width/2)} 0" rpy="0 0 0" />
+        <dynamics damping="0.0" friction="0.0"/>
+        <limit effort= "100" velocity="100"/>
+    </joint>
+    <joint name="base_to_middle_left_wheel" type="continuous">
+        <axis rpy="0 0 0" xyz="0 1 0"/>
+        <parent link="body_link" />
+        <child link="middle_left_wheel" />
+		<origin xyz="0 ${wheel_separation/2 + wheel_width/2} 0" rpy="0 0 0" />
+        <dynamics damping="0.0" friction="0.0"/>
+        <limit effort= "100" velocity="100"/>
+    </joint>
+    <joint name="base_to_middle_right_wheel" type="continuous">
+        <axis rpy="0 0 0" xyz="0 1 0"/>
+        <parent link="body_link" />
+        <child link="middle_right_wheel" />
+		<origin xyz="0 ${-1 * (wheel_separation/2 + wheel_width/2)} 0" rpy="0 0 0" />
+        <dynamics damping="0.0" friction="0.0"/>
+        <limit effort= "100" velocity="100"/>
     </joint>
     <joint name="rear_left_wheel_to_marker" type="fixed">
@@ -206,10 +295,4 @@
         <origin xyz="0.015 0.0175 0" rpy="0 0 0" />
     </joint>
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
Commit message: Added a simple world with geometric objects, added lidar to robot

File: smallbot_description/urdf/smallbot.xacro (robot description, xacro)
@@ -13,5 +13,5 @@
     <xacro:property name="wheel_mass" value="0.2"/>
     <xacro:property name="marker_mass" value="0.0"/>
-    <xacro:property name="inertia" value="1.0"/>
+    <xacro:property name="inertia" value="0.3"/>
     <xacro:property name="PI" value="3.1415926"/>
     <xacro:property name="wheel_ixx" value="${wheel_mass*(3*wheel_radius*wheel_radius+wheel_width*wheel_width)/12}" />
@@ -50,4 +50,31 @@
         <origin xyz="0 0 ${wheel_radius}" rpy="0 0 0"/>
     </joint>
+    <!-- Lidar -->
+    <link name="rplidar_link">
+        <inertial>
+            <origin xyz="0 0 0" rpy="0 0 0" />
+            <mass value="0.1" />
+            <inertia ixx="0.0" ixy="0.0" ixz="0.0" iyy="0.0" iyz="0.0" izz="0.0" />
+        </inertial>
+        <visual>
+            <origin xyz="0 0 0" rpy="0 0 0" />
+            <geometry>
+                <cylinder radius="0.035" length="0.025"/>
+            </geometry>
+            <material name="Blue" />
+        </visual>
+        <collision>
+            <origin xyz="0 0 0" rpy="0 0 0"/>
+            <geometry>
+                <cylinder radius="0.035" length="0.025"/>
+            </geometry>
+        </collision>
+    </link>
+    <joint name="joint_sensor_laser" type="fixed">
+        <origin xyz="0.07 0 0.08" rpy="0 0 0"/>
+        <parent link="body_link"/>
+        <child link="rplidar_link"/>
+    </joint>
+    <!-- Wheels -->
     <link name="rear_left_wheel">
         <visual>
